File: CozyLED/power.kicad_sch (KiCad schematic)
At the start: 7 parts, among them J6 12V Input, U2 LMR16006YQ3

Commit message: Updated Code v0.1
Updates
- Added code for LCD drawings of mode label and triangles to depict button presses (still need actual press drawing)
- Added initial code for mode transition by button hold (2.5 seconds for now)
- Cleaned up some test code
Parts:
- removed C23: 2.2u, Capacitor_SMD:C_0603_1608Metric, symbol Device:C_Small
- removed C24: 100n, Capacitor_SMD:C_0603_1608Metric, symbol Device:C_Small
- removed C25: 10u, Capacitor_SMD:C_0603_1608Metric, symbol Device:C_Small
- removed D2: D_Schottky, Diode_SMD:D_0603_1608Metric, symbol Device:D_Schottky
- removed J6: 12V Input, Connector_BarrelJack:BarrelJack_CUI_PJ-063AH_Horizontal, symbol Connector:Barrel_Jack
- removed L3: 6.8u, Inductor_SMD:L_6.3x6.3_H3, symbol Device:L_Small
- removed U2: LMR16006YQ3, Package_TO_SOT_SMD:SOT-23-6, symbol Regulator_Switching:LMR16006YQ3
Other:
- note removed: "12V IN BARREL JACK CONNECTOR"
- note removed: "12V TO 3.3V DC-DC CONVERTER"
